File: Hardware/PCBA/Pomodoro_V1/Power and USB.kicad_sch (KiCad schematic)
At the start: 0 parts

Commit message: Finalized the schematic, First Draft of the finished Layout
Parts:
- added C25, C28: 1u, Capacitor_SMD:C_0805_2012Metric, symbol Device:C
- added C29: 100n, Capacitor_SMD:C_0805_2012Metric, symbol Device:C
- added C30: 330u, Capacitor_SMD:CP_Elec_6.3x5.8, symbol Device:C_Polarized
- added IC1: LDK120M33R, Package_TO_SOT_SMD:TSOT-23-5, symbol Custom_Parts:LDK120M33R
- added J8: 2171800001, 2171800001:MOLEX_2171800001, symbol 2171800001:2171800001
- added R14, R15, R16: 5k1, Resistor_SMD:R_0805_2012Metric, symbol Device:R
Connections:
- new net: J8.A5 (CC1), R16.1
- new net: IC1.3 (EN), R14.1
- new net: C29.1, IC1.4 (BYP/ADJ/NC)
- new net: J8.B5 (CC2), R15.1
- new net +3V3: C28.1, IC1.5 (VOUT)
- new net +5V: C25.1, C30.1, IC1.1 (VIN), J8.A4B9 (VBUS1), J8.B4A9 (VBUS2), R14.2
- new net GND: C25.2, C28.2, C29.2, C30.2, IC1.2 (GND), J8.A1B12 (GND1), J8.B1A12 (GND2), J8.SH1 (SHIELD1), J8.SH2 (SHIELD2), J8.SH3 (SHIELD3), J8.SH4 (SHIELD4), R15.2, R16.2
- no-connect marks 0 -> 6
Other:
- note added: "LDO 5V -> 3.3V"
- note added: "LDO: 5V -> 3.3V"
- note added: "These 5k1 Pull-Down resistors are necessary for power negotiation on the USB (5V, 3A) https://forum.digikey.com/t/simple-way-to-use-usb-type-c-to-get-5v-at-up-to-3a-15w/7016"
- note added: "USB Connector"

Commit message: Version that was ordered online
Parts:
- C25, C28: Digikey (none) -> https://www.digikey.pt/en/products/detail/nextgen-component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; MPN (none) -> 0805B105K250DC; Part ID 08055C105K4T4A -> (none)
- C29: Digikey (none) -> https://www.digikey.pt/en/products/detail/yageo/CC0805KRX7R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; MPN (none) -> CC0805KRX7R9BB104; Part ID 08051C104KAT4A -> (none)
- C30: Digikey (none) -> https://www.digikey.pt/en/products/detail/w%C3%BCrth-elektr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; MPN (none) -> 875105144010; Part ID 875105144010 -> (none)
- IC1: Digikey (none) -> https://www.digikey.pt/en/products/detail/stmicroelectronic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; MPN (none) -> LDK120M33R; Part ID LDK120M33R -> (none)
- J8: Digikey (none) -> https://www.digikey.pt/en/products/detail/molex/2171800001/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; MANUFACTURER Molex -> (none); MAXIMUM_PACKAGE_HEIGHT 7.78 mm -> (none); MPN (none) -> 2171800001; OPTION MOLEX_CONFIG -> (none); PARTREV A1 -> (none); SNAPEDA_PN 2171800001 -> (none); STANDARD Manufacturer Recommendations -> (none)
- R14, R15, R16: MPN (none) -> CR0805-FX-5101ELF
