File: Hardware/PCBA/Pomodoro_V1/Trigger Btn Lights.kicad_sch (KiCad schematic)
At the start: 6 parts

Commit message: Finalized the schematic, First Draft of the finished Layout
Parts:
- removed C24: 1u, symbol Device:C
- removed C25: 100n, symbol Device:C
- added J10: Conn_01x01_Pin, Connector_PinHeader_2.54mm:PinHeader_1x01_P2.54mm_Vertical, symbol Connector:Conn_01x01_Pin
Connections:
- net at D108.1 (DOUT): now also J10.1 (Pin_1)

Commit message: Version that was ordered online
Parts:
- D105, D106, D107, D108: MPN (none) -> WS2812B-2020
- J10: now not fitted
