File: Hardware/PCBA/Pomodoro_V1/Pomodoro_V1.kicad_pcb (KiCad board)
At the start: 2 copper layers, 107 parts, among them U1 STM32G071RBTx

Commit message: Implemented the Rotary encoder, the buttons, the IMU, Added it to the PCB (All the space constraining elements are now placed)
Parts:
- added D106: WS2812B-2020, LED_SMD:LED_WS2812B-2020_PLCC4_2.0x2.0mm, F.Cu at (158.5, 100.0)
- added D107: WS2812B-2020, LED_SMD:LED_WS2812B-2020_PLCC4_2.0x2.0mm, F.Cu at (150.0, 108.5)
- added D108: WS2812B-2020, LED_SMD:LED_WS2812B-2020_PLCC4_2.0x2.0mm, F.Cu at (141.5, 100.0)
- added REF**: PEC12R-2220F-S0024, Rotary_Encoder:PEC12R-2220F-S0024, B.Cu at (150.0, 67.5)
- added REF**: MOLEX_2171800001, Connector_Molex:MOLEX_2171800001, B.Cu at (150.0, 119.5)
- added U2: LIS2HH12, Package_LGA:LGA-12_2x2mm_P0.5mm, F.Cu at (1.52, 1.52)
- U1: moved to B.Cu
- moved U1 192.5 mm to (131.8, 82.3), turned to 180 degrees
- moved D92 15.7 mm to (145.0, 75.0), turned to 101.25 degrees
- moved D91 12.7 mm to (140.2, 76.4), turned to 112.5 degrees
- moved D93 12.6 mm to (150.0, 84.5), turned to 90 degrees
- moved D94 11.1 mm to (157.8, 86.6), turned to 60 degrees
- moved D90 9.62 mm to (135.8, 78.8), turned to 123.75 degrees
- moved D95 9.58 mm to (163.4, 92.2), turned to 30 degrees
- moved D89 9.29 mm to (132.0, 82.0), turned to 135 degrees
- moved D88 8.97 mm to (128.8, 85.8), turned to 146.25 degrees
- moved D87 8.64 mm to (126.4, 90.2), turned to 157.5 degrees
- moved D105 8.47 mm to (150.0, 91.5), turned to 180 degrees
- moved D86 8.31 mm to (125.0, 95.0), turned to 168.75 degrees
- moved D96 8.02 mm to (165.5, 100.0), turned to 0 degrees
- moved D85 7.98 mm to (124.5, 100.0), turned to 180 degrees
- moved D84 7.65 mm to (125.0, 105.0), turned to -168.75 degrees
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Connections:
- net /µC & Debug Connector/GPIO_OUT (Debug 1) renamed /µC & Debug Connector/GPIO (Debug 1)
- net /µC & Debug Connector/GPIO_OUT (Debug 2) renamed /µC & Debug Connector/GPIO (Debug 2)
- net /µC & Debug Connector/GPIO_OUT (Debug 3) renamed /µC & Debug Connector/GPIO (Debug 3)
- net /µC & Debug Connector/GPIO_OUT (Debug 4) renamed /µC & Debug Connector/GPIO (Debug 4)
- net /µC & Debug Connector/USART1_RX renamed /µC & Debug Connector/USART1_RX (External MCU)
- net /µC & Debug Connector/USART1_TX renamed /µC & Debug Connector/USART1_TX (External MCU)
- net /µC & Debug Connector/USART2_RX renamed /µC & Debug Connector/USART2_RX (Debug)
- net /µC & Debug Connector/USART2_TX renamed /µC & Debug Connector/USART2_TX (Debug)
- net Net-(D104-DOUT) renamed TIM1_CH1 (RgbLed Trigger Btn Light)
- net TIM2_CH1 (Encoder) renamed TIM2_CH1 (Encoder Dial)
- net TIM2_CH2 (Encoder) renamed TIM2_CH2 (Encoder Dial)
- D105 pad 1: unconnected-(D105-DOUT-Pad1) -> Net-(D105-DOUT)
- D90 pad 1: TIM1_CH1 (RgbLed Inner Ring) -> Net-(D90-DOUT)
- D91 pad 3: TIM1_CH1 (RgbLed Inner Ring) -> Net-(D90-DOUT)
- D92 pad 1: Net-(D92-DOUT) -> TIM1_CH1 (RgbLed Inner Ring)
- D93 pad 3: Net-(D92-DOUT) -> TIM1_CH1 (RgbLed Inner Ring)
- U1 pad 29: unconnected-(U1-PB2-Pad29) -> EXTI2 (Accelerometer)
- U1 pad 30: unconnected-(U1-PB10-Pad30) -> EXTI10 (Accelerometer)
- U1 pad 60: /µC & Debug Connector/I2C1_SCL -> I2C1_SCL (Accelerometer)
- U1 pad 61: /µC & Debug Connector/I2C1_SDA -> I2C1_SDA (Accelerometer)
Other:
- board outline added: 78 x 78 mm

Commit message: Finalized the schematic, First Draft of the finished Layout
Parts:
- added C15: 4u7, Capacitor_SMD:C_0805_2012Metric, B.Cu at (168.3, 117.7)
- added C16: 100n, Capacitor_SMD:C_0805_2012Metric, B.Cu at (170.9, 117.7)
- added C17: 100n, Capacitor_SMD:C_0805_2012Metric, B.Cu at (173.0, 117.7)
- added C18: 4u7, Capacitor_SMD:C_0805_2012Metric, B.Cu at (172.5, 112.5)
- added C19: 100n, Capacitor_SMD:C_0805_2012Metric, B.Cu at (170.4, 112.5)
- added C21: 100n, Capacitor_SMD:C_0805_2012Metric, B.Cu at (168.3, 112.5)
- added C22: 100n, Capacitor_SMD:C_0805_2012Metric, B.Cu at (146.1, 90.1)
- added C25: 1u, Capacitor_SMD:C_0805_2012Metric, B.Cu at (158.2, 116.6)
- added C26: 100n, Capacitor_SMD:C_0805_2012Metric, B.Cu at (146.8, 80.5)
- added C27: 100n, Capacitor_SMD:C_0805_2012Metric, B.Cu at (156.6, 80.4)
- added C28: 1u, Capacitor_SMD:C_0805_2012Metric, B.Cu at (164.5, 116.6)
- added C29: 100n, Capacitor_SMD:C_0805_2012Metric, B.Cu at (164.5, 113.1)
- added C30: 330u, Capacitor_SMD:CP_Elec_6.3x5.8, B.Cu at (138.5, 116.0)
- added C31: 100n, Capacitor_SMD:C_0805_2012Metric, B.Cu at (175.6, 86.7)
- added C32: 100n, Capacitor_SMD:C_0805_2012Metric, B.Cu at (148.8, 80.5)
- added D109: LED, Resistor_SMD:R_0603_1608Metric, B.Cu at (182.6, 96.5)
- added IC1: LDK120M33R, Package_TO_SOT_SMD:TSOT-23-5, B.Cu at (161.4, 116.6)
- added J1: Conn_01x02_Pin, Connector_PinHeader_2.54mm:PinHeader_1x02_P2.54mm_Vertical, B.Cu at (122.4, 85.8)
- added J10: Conn_01x01_Pin, Connector_PinHeader_2.54mm:PinHeader_1x01_P2.54mm_Vertical, B.Cu at (138.2, 100.0)
- added J2: Conn_01x10_Pin, Connector:Tag-Connect_TC2050-IDC-NL_2x05_P1.27mm_Vertical, B.Cu at (134.5, 73.2)
- added J3: Conn_01x03_Pin, Connector_PinHeader_2.54mm:PinHeader_1x03_P2.54mm_Vertical, B.Cu at (119.0, 97.5)
- added J4: Conn_01x02_Pin, Connector_PinHeader_2.54mm:PinHeader_1x02_P2.54mm_Vertical, B.Cu at (151.5, 131.0)
- added J5: Conn_01x02_Pin, Connector_PinHeader_2.54mm:PinHeader_1x02_P2.54mm_Vertical, B.Cu at (129.2, 123.0)
- added J6: Conn_01x02_Pin, Connector_PinHeader_2.54mm:PinHeader_1x02_P2.54mm_Vertical, B.Cu at (135.8, 127.6)
- added J7: Conn_01x02_Pin, Connector_PinHeader_2.54mm:PinHeader_1x02_P2.54mm_Vertical, B.Cu at (123.9, 116.8)
- added J9: Conn_01x04_Pin, Connector_PinHeader_2.54mm:PinHeader_1x04_P2.54mm_Vertical, B.Cu at (168.8, 124.9)
- added R1: 5k1, Resistor_SMD:R_0805_2012Metric, B.Cu at (178.4, 112.5)
- added R10: 5k1, Resistor_SMD:R_0805_2012Metric, B.Cu at (148.8, 76.9)
- added R11: 5k1, Resistor_SMD:R_0805_2012Metric, B.Cu at (144.7, 80.5)
- added R12: 5k1, Resistor_SMD:R_0805_2012Metric, B.Cu at (154.5, 80.4)
- added R13: 270, Resistor_SMD:R_0805_2012Metric, B.Cu at (181.3, 92.7)
- added R14: 5k1, Resistor_SMD:R_0805_2012Metric, B.Cu at (158.2, 113.1)
- added R15: 5k1, Resistor_SMD:R_0805_2012Metric, B.Cu at (148.7, 122.4)
- added R16: 5k1, Resistor_SMD:R_0805_2012Metric, B.Cu at (150.7, 122.4)
- added R2: 5k1, Resistor_SMD:R_0805_2012Metric, B.Cu at (180.5, 112.5)
- added R3: 5k1, Resistor_SMD:R_0805_2012Metric, B.Cu at (176.4, 112.5)
- added R4: 5k1, Resistor_SMD:R_0805_2012Metric, B.Cu at (182.5, 112.5)
- added R5: 5k1, Resistor_SMD:R_0805_2012Metric, B.Cu at (144.1, 93.7)
- added R6: 5k1, Resistor_SMD:R_0805_2012Metric, B.Cu at (146.1, 93.7)
- added R7: 5k1, Resistor_SMD:R_0805_2012Metric, B.Cu at (154.5, 76.9)
- added R8: 100, Resistor_SMD:R_0805_2012Metric, B.Cu at (159.8, 69.6)
- added R9: 5k1, Resistor_SMD:R_0805_2012Metric, B.Cu at (144.7, 76.9)
- J8: renamed from REF**; value MOLEX_2171800001 -> 2171800001
- SW1: renamed from REF**; value SW_Cherry_MX_1.00u_PCB -> SW_Push
- U2: moved to B.Cu
- moved U2 211.6 mm to (178.1, 118.2), turned to 180 degrees
- moved U1 43.3 mm to (169.3, 104.0), turned to 90 degrees
- renumbered REF** to S1
Connections:
- D1 pad 3: TIM1_CH1 (RgbLed Outer Ring) -> Net-(D1-DIN)
- D108 pad 1: unconnected-(D108-DOUT-Pad1) -> Net-(D108-DOUT)
- J8 pad A1B12: (no net) -> GND
- J8 pad A4B9: (no net) -> +5V
- J8 pad A5: (no net) -> Net-(J8-CC1)
- J8 pad A6: (no net) -> unconnected-(J8-DP1-PadA6)
- J8 pad A7: (no net) -> unconnected-(J8-DN1-PadA7)
- J8 pad A8: (no net) -> unconnected-(J8-SBU1-PadA8)
- J8 pad B1A12: (no net) -> GND
- J8 pad B4A9: (no net) -> +5V
- J8 pad B5: (no net) -> Net-(J8-CC2)
- J8 pad B6: (no net) -> unconnected-(J8-DP2-PadB6)
- J8 pad B7: (no net) -> unconnected-(J8-DN2-PadB7)
- J8 pad B8: (no net) -> unconnected-(J8-SBU2-PadB8)
- J8 pad SH1: (no net) -> GND
- J8 pad SH2: (no net) -> GND
- J8 pad SH3: (no net) -> GND
- J8 pad SH4: (no net) -> GND
- S1 pad 1: (no net) -> GPIO_IN (Encoder BTN)
- S1 pad 2: (no net) -> GND
- S1 pad A: (no net) -> Net-(S1-CHANNEL_A)
- S1 pad B: (no net) -> Net-(S1-CHANNEL_B)
- S1 pad C: (no net) -> GND
- S1 pad S1: (no net) -> GND
- S1 pad S2: (no net) -> GND
- SW1 pad 1: (no net) -> GND
- SW1 pad 2: (no net) -> Net-(R5-Pad2)
- U1 pad 29: EXTI2 (Accelerometer) -> unconnected-(U1-PB2-Pad29)
- U1 pad 30: EXTI10 (Accelerometer) -> unconnected-(U1-PB10-Pad30)
- U1 pad 36: TIM1_CH1 (RgbLed) -> TIM1_CH1 (RgbLed Outer Ring)
- U1 pad 62: unconnected-(U1-PB8-Pad62) -> EXTI8 (Accelerometer)
- U1 pad 63: unconnected-(U1-PB9-Pad63) -> EXTI9 (Accelerometer)
- U2 pad 11: EXTI10 (Accelerometer) -> EXTI9 (Accelerometer)
- U2 pad 12: EXTI2 (Accelerometer) -> EXTI8 (Accelerometer)
Routing:
- net GND: track 0.00 -> 166.6 mm, vias 0 -> 121
- net +5V: track 0.00 -> 165.7 mm, vias 0 -> 116
- net /µC & Debug Connector/GPIO (Debug 1): track 0.00 -> 148.0 mm, vias 0 -> 4
- net /µC & Debug Connector/GPIO (Debug 2): track 0.00 -> 145.7 mm, vias 0 -> 4
- net +3V3: track 0.00 -> 144.7 mm, vias 0 -> 11
- net /µC & Debug Connector/NRST: track 0.00 -> 138.5 mm, vias 0 -> 5
- net /µC & Debug Connector/GPIO (Debug 4): track 0.00 -> 115.9 mm, vias 0 -> 6
- net /µC & Debug Connector/SWCLK: track 0.00 -> 114.0 mm, vias 0 -> 6
- net /µC & Debug Connector/GPIO (Debug 3): track 0.00 -> 112.5 mm, vias 0 -> 6
- net /µC & Debug Connector/USART2_TX (Debug): track 0.00 -> 105.7 mm, vias 0 -> 4
- net /µC & Debug Connector/USART2_RX (Debug): track 0.00 -> 105.6 mm, vias 0 -> 6
- net /µC & Debug Connector/SWDIO: track 0.00 -> 104.4 mm, vias 0 -> 4
- net GPIO_IN (Encoder BTN): track 0.00 -> 58.7 mm, vias 0 -> 4
- net GPIO_IN (Trigger Btn): track 0.00 -> 40.1 mm, vias 0 -> 4
- net TIM2_CH1 (Encoder Dial): track 0.00 -> 37.2 mm
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- added copper zone on F.Cu, net +5V
- added copper zone on B.Cu, net GND

Commit message: Rerouted the layout
Parts:
- moved C31 30.0 mm to (161.3, 113.1)
- moved C22 21.4 mm to (158.2, 107.8)
- moved R5 17.3 mm to (154.1, 107.8)
- moved R6 17.3 mm to (156.1, 107.8)
- moved R13 16.4 mm to (180.5, 109.1), turned to 90 degrees
- moved R8 8.38 mm to (167.0, 74.0)
- moved D109 7.41 mm to (180.5, 103.6), turned to -90 degrees
- moved J3 5.05 mm to (119.0, 102.5), turned to 0 degrees
- moved U2 1.92 mm to (176.7, 116.8)
Routing:
- net /µC & Debug Connector/GPIO (Debug 1): track 148.0 -> 97.3 mm, vias 4 -> 2
- net /µC & Debug Connector/GPIO (Debug 2): track 145.7 -> 95.5 mm, vias 4 -> 2
- net /µC & Debug Connector/GPIO (Debug 4): track 115.9 -> 73.2 mm, vias 6 -> 2
- net /µC & Debug Connector/NRST: track 138.5 -> 96.0 mm, vias 5 -> 3
- net /µC & Debug Connector/SWCLK: track 114.0 -> 77.9 mm, vias 6 -> 2
- net GND: track 166.6 -> 201.6 mm, vias 121 -> 291
- net /µC & Debug Connector/GPIO (Debug 3): track 112.5 -> 78.2 mm, vias 6 -> 2
- net +5V: track 165.7 -> 136.5 mm, vias 116 -> 276
- net GPIO_IN (Trigger Btn): track 40.1 -> 19.3 mm, vias 4 -> 2
- net Net-(R5-Pad2): track 4.93 -> 23.8 mm, vias 0 -> 2
- net /µC & Debug Connector/USART2_TX (Debug): track 105.7 -> 87.5 mm, vias 4 -> 3
- net /µC & Debug Connector/SWDIO: track 104.4 -> 87.9 mm, vias 4 -> 2
- net /µC & Debug Connector/USART2_RX (Debug): track 105.6 -> 91.8 mm, vias 6 -> 3
- net TIM2_CH1 (Encoder Dial): track 37.2 -> 48.3 mm, vias 0 -> 3
- net +3V3: track 144.7 -> 154.3 mm, vias 11 -> 6
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- added copper zone on B.Cu, net +5V
- added copper zone on In2.Cu, net +5V
- added copper zone on F.Cu, net GND
- added copper zone on In1.Cu, net GND
- removed copper zone on F.Cu, net +5V
- removed copper zone on B.Cu, net GND
Other:
- copper layers 2 -> 4
- board text added: "3.3V"
- board text added: "5V"
- board text added: "Dbg 1"
- board text added: "Dbg 2"
- board text added: "Dbg 3"
- board text added: "Dbg 4"
- board text added: "GND"
- board text added: "NRST"
- board text added: "SWCLK"
- board text added: "SWDIO"
- board text added: "UART1 RX"
- board text added: "UART1 TX"
- board text added: "UART2 RX"
- board text added: "UART2 TX"

Commit message: Version that was ordered online
Parts:
- C15, C18: value 4u7 -> 1u

Commit message: Minor refactoring on the RGBLED Driver, Changed the nominalPomodoro Script a bit, Added some dimensions into Kicad
Changed lines of the file:
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@@
 		)
 		(fp_line
-			(start -1.520001 -1.25)
+			(start -1.520002 -1.25)
 			(end -1.52 1.25)
 			(stroke
@@
 		(fp_line
 			(start -1.52 1.25)
-			(end 1.520001 1.25)
+			(end 1.520002 1.25)
 			(stroke
 				(width 0.05)
@@
 		(fp_line
 			(start 1.52 -1.25)
-			(end -1.520001 -1.25)
+			(end -1.520002 -1.25)
 			(stroke
 				(width 0.05)
@@
 		)
 		(fp_line
-			(start 1.520001 1.25)
+			(start 1.520002 1.25)
 			(end 1.52 -1.25)
 			(stroke
@@
 		)
 		(fp_line
-			(start 1.520001 1.25)
+			(start 1.520002 1.25)
 			(end 1.52 -1.25)
 			(stroke
@@
 		(fp_line
 			(start 1.52 -1.25)
-			(end -1.520001 -1.25)
+			(end -1.520002 -1.25)
 			(stroke
 				(width 0.05)
@@
 		(fp_line
 			(start -1.52 1.25)
-			(end 1.520001 1.25)
+			(end 1.520002 1.25)
 			(stroke
 				(width 0.05)
@@
 		)
 		(fp_line
-			(start -1.520001 -1.25)
+			(start -1.520002 -1.25)
 			(end -1.52 1.25)
 			(stroke
@@
 		(fp_line
 			(start 1.52 -1.25)
-			(end -1.520001 -1.25)
+			(end -1.520002 -1.25)
 			(stroke
 				(width 0.05)
@@
 		)
 		(fp_line
-			(start -1.520001 -1.25)
+			(start -1.520002 -1.25)
 			(end -1.52 1.25)
 			(stroke
@@
 		)
 		(fp_line
-			(start 1.520001 1.25)
+			(start 1.520002 1.25)
 			(end 1.52 -1.25)
 			(stroke
@@
 		(fp_line
 			(start -1.52 1.25)
-			(end 1.520001 1.25)
+			(end 1.520002 1.25)
 			(stroke
 				(width 0.05)
@@
 		(fp_circle
 			(center -1.8 -1)
-			(end -1.7 -1.000001)
+			(end -1.7 -1.000002)
 			(stroke
 				(width 0.1)
@@
 		)
 		(fp_line
-			(start -0.550001 -1)
+			(start -0.550002 -1)
 			(end -1.1 -0.45)
 			(stroke
@@
 		(fp_line
 			(start 1.1 -1)
-			(end -0.550001 -1)
+			(end -0.550002 -1)
 			(stroke
 				(width 0.1)
@@
 		(fp_line
 			(start -1.52 -1.25)
-			(end -1.520001 1.25)
+			(end -1.520002 1.25)
 			(stroke
 				(width 0.05)
@@
 		)
 		(fp_line
-			(start 1.520001 -1.25)
+			(start 1.520002 -1.25)
 			(end -1.52 -1.25)
 			(stroke
@@
 		)
 		(fp_line
-			(start -1.520001 1.25)
+			(start -1.520002 1.25)
 			(end 1.52 1.25)
 			(stroke
@@
 		(fp_line
 			(start 1.52 1.25)
-			(end 1.520001 -1.25)
+			(end 1.520002 -1.25)
 			(stroke
 				(width 0.05)
@@
 		)
 		(fp_line
-			(start 1.520001 -1.25)
+			(start 1.520002 -1.25)
 			(end -1.52 -1.25)
 			(stroke
@@
 		(fp_line
 			(start 1.52 1.25)
-			(end 1.520001 -1.25)
+			(end 1.520002 -1.25)
 			(stroke
 				(width 0.05)
@@
 		(fp_line
 			(start -1.52 -1.25)
-			(end -1.520001 1.25)
+			(end -1.520002 1.25)
 			(stroke
 				(width 0.05)
@@
 		)
 		(fp_line
-			(start -1.520001 1.25)
+			(start -1.520002 1.25)
 			(end 1.52 1.25)
 			(stroke
@@
 		(fp_circle
 			(center -1.8 -1)
-			(end -1.7 -1.000001)
+			(end -1.7 -1.000002)
 			(stroke
 				(width 0.1)
@@
 		(fp_line
 			(start 1.1 -1)
-			(end -0.550001 -1)
+			(end -0.550002 -1)
 			(stroke
 				(width 0.1)
@@
 		)
 		(fp_line
-			(start -0.550001 -1)
+			(start -0.550002 -1)
 			(end -1.1 -0.45)
 			(stroke
@@
 		(fp_line
 			(start 1.52 1.25)
-			(end 1.520001 -1.25)
+			(end 1.520002 -1.25)
 			(stroke
 				(width 0.05)
@@
 		)
 		(fp_line
-			(start -1.520001 1.25)
+			(start -1.520002 1.25)
 			(end 1.52 1.25)
 			(stroke
@@
 		)
 		(fp_line
-			(start 1.520001 -1.25)
+			(start 1.520002 -1.25)
 			(end -1.52 -1.25)
 			(stroke
@@
 		(fp_line
 			(start -1.52 -1.25)
-			(end -1.520001 1.25)
+			(end -1.520002 1.25)
 			(stroke
 				(width 0.05)
@@
 		(fp_line
 			(start -1.52 1.25)
-			(end 1.520001 1.25)
+			(end 1.520002 1.25)
 			(stroke
 				(width 0.05)
@@
 		)
 		(fp_line
-			(start 1.520001 1.25)
+			(start 1.520002 1.25)
 			(end 1.52 -1.25)
 			(stroke
@@
 		)
 		(fp_line
-			(start -1.520001 -1.25)
+			(start -1.520002 -1.25)
 			(end -1.52 1.25)
 			(stroke
@@
 		(fp_line
 			(start 1.52 -1.25)
-			(end -1.520001 -1.25)
+			(end -1.520002 -1.25)
 			(stroke
 				(width 0.05)
@@
 		(fp_circle
 			(center -1.8 -1)
-			(end -1.7 -1.000001)
+			(end -1.7 -1.000002)
 			(stroke
 				(width 0.1)
@@
 		)
 		(fp_line
-			(start -0.550001 -1)
+			(start -0.550002 -1)
 			(end -1.1 -0.45)
 			(stroke
@@
 		(fp_line
 			(start 1.1 -1)
-			(end -0.550001 -1)
+			(end -0.550002 -1)
 			(stroke
 				(width 0.1)
@@
 		(fp_circle
 			(center -1.8 -1)
-			(end -1.7 -1.000001)
+			(end -1.7 -1.000002)
 			(stroke
 				(width 0.1)
@@
 		(fp_line
 			(start 1.1 -1)
-			(end -0.550001 -1)
+			(end -0.550002 -1)
 			(stroke
 				(width 0.1)
@@
 		)
 		(fp_line
-			(start -0.550001 -1)
+			(start -0.550002 -1)
 			(end -1.1 -0.45)
 			(stroke
@@
 		)
 		(fp_line
-			(start -1.520001 1.25)
+			(start -1.520002 1.25)
 			(end 1.52 1.25)
 			(stroke
@@
 		(fp_line
 			(start -1.52 -1.25)
-			(end -1.520001 1.25)
+			(end -1.520002 1.25)
 			(stroke
 				(width 0.05)
@@
 		(fp_line
 			(start 1.52 1.25)
-			(end 1.520001 -1.25)
+			(end 1.520002 -1.25)
 			(stroke
 				(width 0.05)
@@
 		)
 		(fp_line
-			(start 1.520001 -1.25)
+			(start 1.520002 -1.25)
 			(end -1.52 -1.25)
 			(stroke
@@
 		(tags "resistor")
 		(property "Reference" "R13"
-			(at 0 1.65 270)
+			(at 0 1.65 -90)
 			(layer "B.SilkS")
 			(hide yes)
@@
 		)
 		(property "Value" "270"
-			(at 0 -1.65 270)
+			(at 0 -1.65 -90)
 			(layer "B.Fab")
 			(effects
@@
 		)
 		(fp_text user "${REFERENCE}"
-			(at 0 0 270)
+			(at 0 0 -90)
 			(layer "B.Fab")
 			(effects
@@
 		(tags "Through hole pin header THT 1x03 2.54mm single row")
 		(property "Reference" "J3"
-			(at 0 2.33 360)
+			(at 0 2.33 0)
 			(layer "B.SilkS")
 			(hide yes)
@@
 		)
 		(property "Value" "Conn_01x03_Pin"
-			(at 0 -7.41 360)
+			(at 0 -7.41 0)
 			(layer "B.Fab")
 			(hide yes)
@@
 		)
 	)
+	(dimension
+		(type aligned)
+		(layer "Dwgs.User")
+		(pts
+			(xy 139 100) (xy 161 100)
+		)
+		(height -37.33)
+		(gr_text "22.0000 mm"
+			(at 150 61.52 0)
+			(layer "Dwgs.User")
+			(effects
+				(font
+					(size 1 1)
+					(thickness 0.15)
+				)
+			)
+		)
+		(format
+			(prefix "")
+			(suffix "")
+			(units 3)
+			(units_format 1)
+			(precision 4)
+		)
+		(style
+			(thickness 0.1)
+			(arrow_length 1.27)
+			(text_position_mode 0)
+			(extension_height 0.58642)
+			(extension_offset 0.5) keep_text_aligned)
+	)
+	(dimension
+		(type aligned)
+		(layer "Dwgs.User")
+		(pts
+			(xy 109.02 102.58) (xy 191.02 102.58)
+		)
+		(height -50.01)
+		(gr_text "82.0000 mm"
+			(at 150.02 51.42 0)
+			(layer "Dwgs.User")
+			(effects
+				(font
+					(size 1 1)
+					(thickness 0.15)
+				)
+			)
+		)
+		(format
+			(prefix "")
+			(suffix "")
+			(units 3)
+			(units_format 1)
+			(precision 4)
+		)
+		(style
+			(thickness 0.1)
+			(arrow_length 1.27)
+			(text_position_mode 0)
+			(extension_height 0.58642)
+			(extension_offset 0.5) keep_text_aligned)
+	)
+	(dimension
+		(type aligned)
+		(layer "Dwgs.User")
+		(pts
+			(xy 129 100) (xy 171 100)
+		)
+		(height -42.18)
+		(gr_text "42.0000 mm"
+			(at 150 56.67 0)
+			(layer "Dwgs.User")
+			(effects
+				(font
+					(size 1 1)
+					(thickness 0.15)
+				)
+			)
+		)
+		(format
+			(prefix "")
+			(suffix "")
+			(units 3)
+			(units_format 1)
+			(precision 4)
+		)
+		(style
+			(thickness 0.1)
+			(arrow_length 1.27)
+			(text_position_mode 0)
+			(extension_height 0.58642)
+			(extension_offset 0.5) keep_text_aligned)
+	)
+	(dimension
+		(type aligned)
+		(layer "Dwgs.User")
+		(pts
+			(xy 119 99.985) (xy 181 100)
+		)
+		(height -44.443817)
+		(gr_text "62.0000 mm"
+			(at 150.011031 54.398684 359.9861381)
+			(layer "Dwgs.User")
+			(effects
+				(font
+					(size 1 1)
+					(thickness 0.15)
+				)
+			)
+		)
+		(format
+			(prefix "")
+			(suffix "")
+			(units 3)
+			(units_format 1)
+			(precision 4)
+		)
+		(style
+			(thickness 0.1)
+			(arrow_length 1.27)
+			(text_position_mode 0)
+			(extension_height 0.58642)
+			(extension_offset 0.5) keep_text_aligned)
+	)
 	(segment
