File: Hardware/PCBA/Pomodoro_V7/Pomodoro_V7.kicad_pcb (KiCad board)
At the start: 4 copper layers, 76 x 76 mm, 136 parts, among them IC1 ESP32-S2-MINI-2-N4, J1 Conn_01x02_Pin, J10 Conn_01x02_Pin, J11 Conn_01x02_Pin, J12 Conn_01x02_Pin, J13 Conn_01x03_Pin, J14 Conn_01x02_Pin, J15 Conn_01x02_Pin, J2 Conn_01x01_Pin, J3 Conn_01x01_Pin, J4 USB4120-03-C_REVA, J5 Conn_01x02_Pin, J6 Conn_01x02_Pin, J7 Conn_01x05_Pin, J8 Conn_01x02_Pin, J9 Conn_01x02_Pin, U1 LIS2HH12, U2 USBLC6-2SC6, U3 AP2112K-3.3

Commit message: Update on the PCBA
Parts:
- removed TP10: TestPoint, TestPoint:TestPoint_Pad_D1.0mm
- added TP33: TestPoint, TestPoint:TestPoint_Pad_D1.0mm, B.Cu at (36.3, 39.3)
- added TP34: TestPoint, TestPoint:TestPoint_Pad_D1.0mm, B.Cu at (59.3, 64.0)
- added TP35: TestPoint, TestPoint:TestPoint_Pad_D1.0mm, B.Cu at (68.7, 64.0)
- C1: value 10u/16V -> 1u/16V; moved to B.Cu
- C2, C5, C6, C7, C8, C9, J12, J6, J8, J9, JP1, JP2, JP4, R1, R10, R4, R5, R8, R9, TP1, TP11, TP12, TP13, TP14, TP15, TP16, TP17, TP18, TP19, TP2, TP20, TP21, TP22, TP23, TP24, TP25, TP26, TP27, TP28, TP29, TP3, TP30, TP31, TP32, TP4, TP5, TP6, TP7, TP8, TP9, U1, U2, U3: moved to B.Cu
- C3: value 100n/16V -> 10u/16V; moved to B.Cu
- C4: value 1u/16V -> 100n/16V; moved to B.Cu
- J1: value Conn_01x02_Pin -> Conn_01x05_Pin; footprint Connector_PinHeader_2.54mm:PinHeader_1x02_P2.54mm_Horizontal -> Connector_PinHeader_2.54mm:PinHeader_1x05_P2.54mm_Vertical; moved to F.Cu
- J10: footprint Connector_PinHeader_2.54mm:PinHeader_1x02_P2.54mm_Vertical -> Connector_PinHeader_2.54mm:PinHeader_1x02_P2.54mm_Horizontal; moved to B.Cu
- J11: value Conn_01x02_Pin -> USB4120-03-C_REVA; footprint Connector_PinHeader_2.54mm:PinHeader_1x02_P2.54mm_Vertical -> Connector:GCT_USB4120-03-C_REVA; moved to B.Cu
- J13: value Conn_01x03_Pin -> Conn_01x02_Pin; footprint Connector_PinHeader_2.54mm:PinHeader_1x03_P2.54mm_Vertical -> Connector_PinHeader_2.54mm:PinHeader_1x02_P2.54mm_Vertical; moved to B.Cu
- J14, J15: value Conn_01x02_Pin -> Conn_01x01_Pin; footprint Connector_PinHeader_2.54mm:PinHeader_1x02_P2.54mm_Vertical -> Connector_PinHeader_2.54mm:PinHeader_1x01_P2.54mm_Vertical; moved to B.Cu
- J2, J3: value Conn_01x01_Pin -> Conn_01x02_Pin; footprint Connector_PinHeader_2.54mm:PinHeader_1x01_P2.54mm_Vertical -> Connector_PinHeader_2.54mm:PinHeader_1x02_P2.54mm_Vertical; moved to B.Cu
- J4: value USB4120-03-C_REVA -> Conn_01x02_Pin; footprint Connector:GCT_USB4120-03-C_REVA -> Connector_PinHeader_2.54mm:PinHeader_1x02_P2.54mm_Vertical; moved to F.Cu
- J5: value Conn_01x02_Pin -> Conn_01x03_Pin; footprint Connector_PinHeader_2.54mm:PinHeader_1x02_P2.54mm_Vertical -> Connector_PinHeader_2.54mm:PinHeader_1x03_P2.54mm_Vertical; moved to B.Cu
- J7: value Conn_01x05_Pin -> Conn_01x02_Pin; footprint Connector_PinHeader_2.54mm:PinHeader_1x05_P2.54mm_Vertical -> Connector_PinHeader_2.54mm:PinHeader_1x02_P2.54mm_Vertical; moved to B.Cu
- JP3: value SolderJumper_2_Open -> SolderJumper_2_Bridged; footprint Jumper:SolderJumper-2_P1.3mm_Open_RoundedPad1.0x1.5mm -> Jumper:SolderJumper-2_P1.3mm_Bridged2Bar_RoundedPad1.0x1.5mm; moved to B.Cu
- JP5: value SolderJumper_2_Bridged -> SolderJumper_2_Open; footprint Jumper:SolderJumper-2_P1.3mm_Bridged2Bar_RoundedPad1.0x1.5mm -> Jumper:SolderJumper-2_P1.3mm_Open_RoundedPad1.0x1.5mm; moved to B.Cu
- R11: value 5k1(1%) -> 100; moved to B.Cu
- R2: value 100 -> 5k1(1%); moved to B.Cu
- R3: value 10k(1%) -> 5k1(1%); moved to B.Cu
- R6: value 2k 1/20W -> 10k 1/20W
- R7: value 1k(1%) -> 5k1(1%); moved to B.Cu
- moved J11 182.3 mm to (150.0, 130.0), turned to 180 degrees
- moved R10 164.0 mm to (146.8, 123.5), turned to -90 degrees
- moved J10 156.4 mm to (151.3, 80.0), turned to 90 degrees
- moved R9 155.4 mm to (154.0, 123.5), turned to -90 degrees
- moved TP23 150.1 mm to (144.9, 80.0), turned to 180 degrees
- moved TP2 149.8 mm to (131.0, 85.8), turned to 180 degrees
- moved TP1 147.8 mm to (128.8, 82.5), turned to 180 degrees
- moved R4 143.6 mm to (170.2, 96.6)
- moved U2 143.0 mm to (150.0, 123.5)
- moved J12 131.5 mm to (137.3, 70.5), turned to 90 degrees
- moved C1 131.3 mm to (131.0, 82.8), turned to -90 degrees
- moved J1 129.0 mm to (25.1, 52.6)
- moved J2 123.2 mm to (125.2, 79.5), turned to -90 degrees
- moved C2 122.2 mm to (118.5, 87.2)
- moved C3 119.0 mm to (118.5, 85.0)
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Connections:
- C1 pad 1: +3V3 -> /MicroController/ESP32_EN
- C4 pad 1: /MicroController/ESP32_EN -> +3V3
- J1 pad 2: ESP32_Button_Signal -> /MicroController/JTAG_TCK
- J10 pad 1: /MicroController/ESP32_DBG2 -> GND
- J10 pad 2: /MicroController/ESP32_DBG1 -> ESP32_Button_Signal
- J12 pad 1: /MicroController/ESP32_DBG6 -> GND
- J12 pad 2: /MicroController/ESP32_DBG5 -> +3V3
- J13 pad 2: TXD0 -> VBUS
- J14 pad 1: GND -> ESP32_RgbLed_DIN
- J15 pad 1: GND -> Net-(D60-DOUT)
- J2 pad 1: ESP32_RgbLed_DIN -> GND
- J3 pad 1: Net-(D60-DOUT) -> GND
- J5 pad 2: /MicroController/BOOT_OPTION -> TXD0
- J6 pad 1: GND -> /MicroController/ESP32_DBG2
- J6 pad 2: /MicroController/ESP32_EN -> /MicroController/ESP32_DBG1
- J7 pad 1: GND -> /MicroController/ESP32_DBG4
- J7 pad 2: /MicroController/JTAG_TCK -> /MicroController/ESP32_DBG3
- J8 pad 1: I2C_SCL -> /MicroController/ESP32_DBG6
- J8 pad 2: I2C_SDA -> /MicroController/ESP32_DBG5
- J9 pad 2: +5V -> ESP32_Button_Signal
- JP3 pad 1: Net-(D60-DOUT) -> I2C_SDA
- JP3 pad 2: ESP32_RgbLed_DOUT -> /MicroController/ESP32_NOM_I2C_SDA
- JP4 pad 1: I2C_SDA -> /MicroController/ESP32_NOM_I2C_SCL
- JP4 pad 2: /MicroController/ESP32_NOM_I2C_SDA -> I2C_SCL
- JP5 pad 1: /MicroController/ESP32_NOM_I2C_SCL -> Net-(D60-DOUT)
- JP5 pad 2: I2C_SCL -> ESP32_RgbLed_DOUT
- R1 pad 1: ESP32_Button_Signal -> /MicroController/ESP32_EN
- R10 pad 1: I2C_SCL -> GND
- R10 pad 2: +3V3 -> Net-(J11-CC2)
- R11 pad 1: I2C_SDA -> ESP32_RgbLed_DIN
- R11 pad 2: +3V3 -> Net-(D1-DIN)
- R2 pad 1: ESP32_RgbLed_DIN -> I2C_SCL
- R2 pad 2: Net-(D1-DIN) -> +3V3
- R3 pad 1: /MicroController/ESP32_EN -> I2C_SDA
- R4 pad 1: GND -> +3V3
- R4 pad 2: Net-(J4-CC2) -> Net-(R4-Pad2)
- R5 pad 1: GND -> +3V3
- R5 pad 2: Net-(J4-CC1) -> ESP32_Button_Signal
- R6 pad 1: Net-(R6-Pad1) -> Net-(R4-Pad2)
- R7 pad 1: Net-(R6-Pad1) -> +3V3
- R7 pad 2: +3V3 -> Net-(U1-~{CS})
- R8 pad 1: +3V3 -> Net-(U1-SA0/SDO)
- R8 pad 2: Net-(U1-~{CS}) -> GND
- R9 pad 1: Net-(U1-SA0/SDO) -> GND
- R9 pad 2: GND -> Net-(J11-CC1)
- TP1 pad 1: I2C_SDA -> /MicroController/ESP32_EN
- TP11 pad 1: /MicroController/ESP32_EN -> I2C_SDA
- TP12 pad 1: +3V3 -> I2C_SCL
- TP13 pad 1: ESP32_RgbLed_DIN -> /MicroController/ESP32_DBG1
- TP14 pad 1: +5V -> /MicroController/ESP32_DBG2
- TP15 pad 1: +5V -> /MicroController/ESP32_DBG3
- TP16 pad 1: GND -> RXD0
- TP17 pad 1: GND -> /MicroController/ESP32_DBG4
- TP18 pad 1: Net-(D60-DOUT) -> TXD0
- TP19 pad 1: /MicroController/ESP32_DBG1 -> GND
- TP2 pad 1: I2C_SCL -> GND
- TP20 pad 1: /MicroController/ESP32_DBG2 -> /MicroController/ESP32_DBG5
- TP21 pad 1: /MicroController/ESP32_DBG3 -> /MicroController/ESP32_DBG6
- TP22 pad 1: /MicroController/ESP32_DBG4 -> ESP32_ADC_POTI
- TP23 pad 1: /MicroController/ESP32_DBG5 -> ESP32_Button_Signal
- TP24 pad 1: /MicroController/ESP32_DBG6 -> IMU_INT1
- TP25 pad 1: TXD0 -> IMU_INT2
- TP26 pad 1: RXD0 -> ESP32_USB_D-
- TP27 pad 1: GND -> ESP32_USB_D+
- TP28 pad 1: ESP32_Button_Signal -> +3V3
- TP29 pad 1: +3V3 -> GND
- TP3 pad 1: GND -> /MicroController/JTAG_TMS
- TP30 pad 1: ESP32_USB_D- -> VBUS
- TP31 pad 1: ESP32_USB_D+ -> VBUS
- TP4 pad 1: /MicroController/BOOT_OPTION -> /MicroController/JTAG_TDI
- TP5 pad 1: GND -> /MicroController/JTAG_TDO
- TP6 pad 1: /MicroController/JTAG_TMS -> /MicroController/JTAG_TCK
- TP7 pad 1: /MicroController/JTAG_TDI -> GND
- TP8 pad 1: /MicroController/JTAG_TDO -> /MicroController/BOOT_OPTION
- TP9 pad 1: /MicroController/JTAG_TCK -> GND
Routing:
- net ESP32_Button_Signal: track 0.00 -> 7.50 mm
- net GND: vias 120 -> 121
