File: Hardware/PCBA/Pomodoro_V7/Pomodoro_V7.kicad_pcb (KiCad board)
At the start: 4 copper layers, 76 x 76 mm, 139 parts, among them IC1 ESP32-S2-MINI-2-N4, J1 Conn_01x05_Pin, J10 Conn_01x02_Pin, J11 USB4120-03-C_REVA, J12 Conn_01x02_Pin, J13 Conn_01x02_Pin, J14 Conn_01x01_Pin, J15 Conn_01x01_Pin, J2 Conn_01x02_Pin, J3 Conn_01x02_Pin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

Commit message: Updated the PCBA Files
Parts:
- removed REF** (x4): Fiducial_0.75mm_Mask1.5mm, Fiducial:Fiducial_0.75mm_Mask1.5mm
- C1, C5, C8, C9: value 1u/16V -> 1u/16V+/X5R
- C2, C3: value 10u/16V -> 10u/16V+/X5R
- C4, C6, C7: value 100n/16V -> 100n/16V+/X5R
- R11: value 100 -> 100R(1%)
- U1: footprint Package_LGA:LGA-12_2x2mm_P0.5mm -> Package_LGA:Kionix_LGA-12_2x2mm_P0.5mm_LayoutBorder2x4y
Routing:
- net GND: track 104.3 -> 105.2 mm
Other:
- board size 76 x 76 mm -> 75.1 x 75.1 mm
